Commit message: Add files via upload

File: ros2_ws/src/ros2_workspace/my_robot_description/urdf/gazebo_plugin.xacro (robot description, xacro)
@@ -1,8 +1,4 @@
 <?xml version="1.0"?>
 <robot xmlns:xacro="http://www.ros.org/wiki/xacro">
-    <gazebo reference="caster_wheel_link">
-        <mu>0.1</mu>
-        <mu2>0.1</mu2>
-    </gazebo>
     <gazebo>
         <plugin filename="gz-sim-diff-drive-system" name="gz::sim::systems::DiffDrive">
@@ -21,79 +17,3 @@
         </plugin>
     </gazebo>
-    <gazebo reference="lidar_link">
-        <sensor name="gpu_lidar" type="gpu_lidar">
-            <topic>scan</topic>
-            <update_rate>10</update_rate>
-            <gz_frame_id>lidar_link</gz_frame_id>
-            <lidar>
-                <scan>
-                    <horizontal>
-                        <samples>720</samples>
-                        <resolution>1</resolution>
-                        <min_angle>-3.1416</min_angle>
-                        <max_angle>3.1416</max_angle>
-                    </horizontal>
-                    <vertical>
-                        <samples>1</samples>
-                        <resolution>1</resolution>
-                        <min_angle>0</min_angle>
-                        <max_angle>0</max_angle>
-                    </vertical>
-                </scan>
-                <range>
-                    <min>0.08</min>
-                    <max>10.0</max>
-                    <resolution>0.01</resolution>
-                </range>
-                <!-- <noise>
-                    <type>gaussian</type>
-                    <mean>0.0</mean>
-                    <stddev>0.01</stddev>
-                </noise> -->
-                <frame_id>lidar_link</frame_id>
-            </lidar>
-            <alwaysOn>true</alwaysOn>
-            <visualize>true</visualize>
-        </sensor>
-    </gazebo>
-    <gazebo reference="imu_link">
-        <sensor name="imu" type="imu">
-            <always_on>1</always_on>
-            <update_rate>50</update_rate>
-            <visualize>true</visualize>
-            <topic>imu</topic>
-            <enable_metrics>true</enable_metrics>
-            <gz_frame_id>imu_link</gz_frame_id>
-        </sensor>
-    </gazebo>
-    <gazebo reference="camera_link">
-        <sensor name="camera" type="camera">
-            <camera>
-                <horizontal_fov>1.3962634</horizontal_fov>
-                <image>
-                    <width>640</width>
-                    <height>480</height>
-                    <format>R8G8B8</format>
-                </image>
-                <clip>
-                    <near>0.1</near>
-                    <far>15</far>
-                </clip>
-                <noise>
-                    <type>gaussian</type>
-                    <!-- Noise is sampled independently per pixel on each frame.
-                        That pixel's noise value is added to each of its color
-                        channels, which at that point lie in the range [0,1]. -->
-                    <mean>0.0</mean>
-                    <stddev>0.007</stddev>
-                </noise>
-                <optical_frame_id>camera_link_optical</optical_frame_id>
-                <camera_info_topic>camera/camera_info</camera_info_topic>
-            </camera>
-            <always_on>1</always_on>
-            <update_rate>20</update_rate>
-            <visualize>true</visualize>
-            <topic>camera/image_raw</topic>
-        </sensor>
-    </gazebo>
 </robot>

File: ros2_ws/src/ros2_workspace/my_robot_description/urdf/my_robot_ros2_control.urdf.xacro (robot description, xacro)
@@ -6,7 +6,5 @@
     <xacro:include filename="imu.xacro"/>
     <xacro:include filename="camera.xacro"/>
-    <xacro:include filename="gazebo_plugin.xacro"/>
     <xacro:include filename="gazebo_sensor_plugin.xacro"/>
-    <xacro:include filename="ros2_control.xacro"/>
     <joint name="lidar_joint" type="fixed">
         <origin xyz="0.0 0.0 ${base_height}" rpy="0.0 0.0 0.0"/>
@@ -24,3 +22,24 @@
         <child link="camera_link"/>
     </joint>
+    <ros2_control name="MyRobotHardwareInterface" type="system">
+        <hardware>
+            <plugin>gz_ros2_control/GazeboSimSystem</plugin>
+            <param name="calculate_dynamics">true</param>
+        </hardware>
+        <joint name="left_wheel_joint">
+            <command_interface name="velocity"/>
+            <state_interface name="position"/>
+            <state_interface name="velocity"/>
+        </joint>
+        <joint name="right_wheel_joint">
+            <command_interface name="velocity"/>
+            <state_interface name="position"/>
+            <state_interface name="velocity"/>
+        </joint>
+    </ros2_control>
+    <gazebo>
+        <plugin filename="gz_ros2_control-system" name="gz_ros2_control::GazeboSimROS2ControlPlugin">
+            <parameters>$(find my_robot_bringup)/config/my_robot_controllers.yaml</parameters>
+        </plugin>
+    </gazebo>
 </robot>
